File: Design/RFH-2.sch (EAGLE design)
At the start: 37 parts

Commit message: Revision B
* Fixed the push-button pinout
* Now makes extensive use of ground plane
* Rewired the board
* Larger holes, suitable for a screw, with symmetrical holes at the
* board edges
* A through-the-hole pad for the signal input
* Added a few centimeters more to accomodate the $ABOVE changes
* And that's it folks!
Parts:
- removed PAD1, PAD2: (no value), wirepad:SMD5
- added TP1, TP2: TPPAD1-20Y, testpad:TPPAD1-20Y
Connections:
- removed net N$2: C1.1, PAD1.P, R1.2, R11.2, R13.2, R16.2, R17.2, R20.2, R21.2, R23.2, R3.2, R5.2, R7.2, R9.2
- new net GNDA: C1.1, R1.2, R11.2, R13.2, R16.2, R17.2, R20.2, R21.2, R23.2, R3.2, R5.2, R7.2, R9.2, TP1.TP
- net N$1: now also TP2.TP; no longer PAD2.P
- net N$10: no longer 2.S1
- net N$11: no longer 3.S1
- net N$12: no longer 4.S1
- net N$13: no longer 5.S1
- net N$14: no longer MEM.S1
- net N$3: no longer LEFT.S1
- net N$4: no longer UP.S1
- net N$5: no longer RIGHT.S1
- net N$6: no longer P/B.S1
- net N$7: no longer DOWN.S1
- net N$8: no longer 1.S1
- net N$9: no longer DEC.S1

Commit message: Schematic: Fixes #1
https://github.com/jgedmond pointed a flipped Down Arrow and F/B
button. Thanks for reporting it!
Parts:
- removed R23: 1k5, rcl:R-US_0309/10
- removed R24: 24k, rcl:R-US_0309/10
- added R15: 6k8, rcl:R-US_0309/10
- R16: value 6k8 -> 12k
- R19: value 13k -> 12K
- R20: value 12k -> 1k5
- R21: value 3k9 -> 24k
- renumbered R22 to R19
Connections:
- removed net N$19: R19.2, R21.1
- net GNDA: now also R15.2, R19.2; no longer R21.2, R23.2
- net N$26: now also R20.1, R21.2; no longer R23.1, R24.2
- net N$4: now also R15.1; no longer R16.1
- net N$5: now also R16.1; no longer R18.1
- net N$6: now also R18.1; no longer R20.1
- net N$9: now also R21.1; no longer R24.1
Other:
- moved on the sheet: R16, R17, R18, R20, R21
